Commit message: Port irobot_hand_description to ROS 2 (ament_cmake)
- content identical between src/drcsim and vigir_atlas_common reference copy
  (vigir_atlas_common only adds redundant .obj mesh exports); converted the
  existing files in place
- catkin -> ament_cmake, package.xml format 2 -> 3 (correct element order
  from the start this time: license/url before author)
- install(DIRECTORY/FILES) to share/<pkg>, dropped make_standalone_models(),
  added GZ_SIM_RESOURCE_PATH environment hook (same rationale as
  multisense_sl_description)
- removed dead nested CMakeLists.txt files (launch/, meshes/) -- unreferenced
  by the new top-level install(DIRECTORY ...)
- converted launch/upload.launch (ROS 1 roslaunch XML, unused by any other
  package in this repo) to launch/upload.launch.py: a robot_state_publisher
  node fed by xacro via a Command substitution
- fixed a real modeling gap: irobot_hand_description.urdf.xacro instantiates
  the irobot_hand macro with parent="world" but never defined a <link
  name="world"/>, so joints referenced an undefined link. Confirmed via
  grep that robotiq_hand_description.urdf.xacro already follows the
  link-name=world + parent=world convention elsewhere in this repo; added
  the missing <link name="world"/> here to match
- added a pytest test (same structural URDF validation as
  multisense_sl_description) covering both top-level xacro files

File: irobot_hand_description/robots/irobot_hand_description.urdf.xacro (robot description, xacro)
@@ -1,4 +1,5 @@
 <robot xmlns:xacro="http://www.ros.org/wiki/xacro" name="atlas" >
   <xacro:include filename="$(find irobot_hand_description)/urdf/irobot_hand.urdf.xacro" />
+  <link name="world"/>
   <xacro:irobot_hand side="left" parent="world" reflect="-1">
     <origin rpy="0 0 0" xyz="0 0 1.0"/>
