Commit message: Port atlas_description to ROS 2 Jazzy (ament_cmake)
Convert package.xml/CMakeLists.txt from catkin to ament_cmake, drop the
make_standalone_models()/URDF_helpers.cmake GAZEBO_MODEL_PATH machinery
in favor of an ament_environment_hooks() GZ_SIM_RESOURCE_PATH hook, and
remove the dead nested meshes/materials CMakeLists.txt files.

Fix real pre-existing left/right mirroring bugs found by diffing against
vigir_atlas_common's fork (used as reference per project convention):
atlas_v4/v5_robotiq_hands.urdf.xacro and atlas_v4/v5_sandia_hands.urdf.xacro
had the left-hand mount origin using the same xyz/rpy signs as the right
hand instead of the mirrored ones (the base non-versioned
atlas_robotiq_hands.urdf.xacro already had this right, confirming it was
a copy-paste bug in the v4/v5 variants). atlas_v4_no_wry2_simple_shapes.urdf
had l_clav referencing r_clav.dae and other left-side links carrying
right-side offsets/mesh paths -- replaced with vigir's corrected skeleton,
same for atlas_v5_simple_shapes.urdf.

Add a pytest that runs xacro on all 25 top-level robots/*.urdf.xacro
variants and structurally validates the resulting URDF, following the
established description-package test pattern.

File: atlas_description/robots/atlas_v4_robotiq_hands.urdf.xacro (robot description, xacro)
@@ -5,5 +5,5 @@
   to mach the values in your actual robot. -->
   <xacro:robotiq_hand prefix="l_" parent="l_hand" reflect="-1">
-    <origin rpy="3.14159 3.14159 0" xyz="-0.00125 -0.17 0.01"/>
+    <origin rpy="3.14159 3.14159 3.14159" xyz="-0.00125 0.17 0.01"/>
   </xacro:robotiq_hand>
   <xacro:robotiq_hand prefix="r_" parent="r_hand" reflect="1">

File: atlas_description/robots/atlas_v4_sandia_hands.urdf.xacro (robot description, xacro)
@@ -6,5 +6,5 @@
   </xacro:sandia_hand>
   <xacro:sandia_hand side="left" parent="l_hand" reflect="-1" joint_type="revolute" thumb_angle="0">
-    <origin xyz="0.00179  -0.13516 0.01176" rpy="0 0  -1.57079"/>
+    <origin xyz="0.00179  0.13516 0.01176" rpy="0 0  1.57079"/>
   </xacro:sandia_hand>
   <xacro:include filename="$(find atlas_description)/urdf/atlas_v4.gazebo" />

File: atlas_description/robots/atlas_v5_robotiq_hands.urdf.xacro (robot description, xacro)
@@ -5,5 +5,5 @@
   to mach the values in your actual robot. -->
   <xacro:robotiq_hand prefix="l_" parent="l_hand" reflect="-1">
-    <origin rpy="3.14159 3.14159 0" xyz="-0.00125 -0.17 0.01"/>
+    <origin rpy="3.14159 3.14159 3.14159" xyz="-0.00125 0.17 0.01"/>
   </xacro:robotiq_hand>
   <xacro:robotiq_hand prefix="r_" parent="r_hand" reflect="1">

File: atlas_description/robots/atlas_v5_sandia_hands.urdf.xacro (robot description, xacro)
@@ -6,5 +6,5 @@
   </xacro:sandia_hand>
   <xacro:sandia_hand side="left" parent="l_hand" reflect="-1" joint_type="revolute" thumb_angle="0">
-    <origin xyz="0.00179  -0.13516 0.01176" rpy="0 0  -1.57079"/>
+    <origin xyz="0.00179  0.13516 0.01176" rpy="0 0  1.57079"/>
   </xacro:sandia_hand>
   <xacro:include filename="$(find atlas_description)/urdf/atlas_v5.gazebo" />

File: atlas_description/urdf/atlas_v4_no_wry2_simple_shapes.urdf (robot description, URDF)
Before this commit: robot drc_skeleton, 32 links, 32 joints
Links:
- link l_clav: geometry collision box size=0.1 0.07 0.072; collision cylinder length=0.1525 radius=0.0555
- link l_foot: geometry collision box size=${0.26-0.033} ${0.124887+0.009} 0.05; collision box size=0.1 ${0.08} 0.02
- link l_hand: geometry collision box size=0.13 0.09 0.07; collision cylinder length=0.05 radius=0.03
- link l_larm: geometry collision box size=0.135 0.15 0.06; collision cylinder length=0.125 radius=0.045
- link l_scap: geometry collision box size=0.02 0.029 0.018; collision box size=0.028 0.090 0.05
- link l_uarm: geometry collision box size=0.05 0.07 0.15; collision cylinder length=0.11 radius=0.065
- link l_ufarm: geometry collision box size=0.135 0.1 0.045; collision cylinder length=0.125 radius=0.045
- link r_foot: geometry collision box size=${0.26-0.033} ${0.124887+0.009} 0.05; collision box size=0.1 ${0.08} 0.02
Joints:
- joint l_arm_elx: axis -1.0 -0.0 -0.0 -> 1 0 0; origin xyz=0 -0.119 0.0092 rpy=0 -0 0 -> xyz=0 0.119 0.0092 rpy=0 -0 0
- joint l_arm_ely: axis -0.0 -1.0 -0.0 -> 0 1 0; origin xyz=0 -0.187 -0.016 rpy=0 -0 0 -> xyz=0 0.187 -0.016 rpy=0 -0 0
- joint l_arm_shx: axis -1.0 -0.0 -0.0 -> 1 0 0; origin xyz=0 -0.11 -0.245 rpy=0 -0 0 -> xyz=0 0.11 -0.245 rpy=0 -0 0
- joint l_arm_shz: origin xyz=0.1406 0.2256 0.4776 rpy=0 0 3.14159265359 -> xyz=0.1406 0.2256 0.4776 rpy=0 -0 0
- joint l_arm_wrx: origin xyz=0 -0.119 0.0092 rpy=0 -0 0 -> xyz=0 0.119 0.0092 rpy=0 -0 0
- joint l_arm_wry: axis -0.0 -1.0 -0.0 -> 0 1 0; origin xyz=0 -0.187 -0.0092 rpy=0 3.14159265359 0 -> xyz=0 0.187 -0.0092 rpy=0 -0 0

File: atlas_description/urdf/atlas_v5_simple_shapes.urdf (robot description, URDF)
Before this commit: robot drc_skeleton, 34 links, 34 joints
Links:
- link utorso: geometry collision box size=0.13 0.50 0.10; collision box size=0.2 0.18 0.10
Joints:
- joint l_arm_wry2: axis 0 1 0 -> 0 -1 0
