Commit message: Omnidirectional harness walking, teleop, kicks, Sandia hands; fix red RViz model
atlas_walking_demo:
- harness_gait.py is velocity-driven (forward/back, side-step, turn, curve)
  with full 3D leg IK (hip yaw/roll/pitch, knee, ankle pitch/roll); stance
  feet move exactly opposite the pelvis, swing feet land at ground speed.
- walk_keyboard.py: game-style keys, speed steps, Twist on
  atlas_walk/cmd_vel, Sandia gripper open/close, and kicks via gz
  ApplyLinkWrench. Pure helpers in teleop_extras.py, all unit-tested.

drcsim_gazebo: hands:=sandia (default) | none. One extra
robot_state_publisher per extra joint-state topic (MultiSense lidar, both
hands) -- the missing hokuyo_joint TF is what turned RViz's RobotModel red.

Sandia hands under gz-sim: plugin tags converted; fixed joints renamed so
they no longer clash with link names in SDFormat's frame graph;
SandiaHandPlugin now gets its finger gains via RosNodeOptionsFromEnv();
dead Classic plugins dropped. VRCPlugin logs spawn SDF errors once instead
of aborting on a re-declared parameter, and its harness damps toward the
commanded yaw rate. atlas.world loads ApplyLinkWrench.

Tests: atlas_walking_demo 56, drcsim_gazebo 14, drcsim_gazebo_ros_plugins
160, sandia_hand_description 24, atlas_description 37,
drcsim_model_resources 120 -- 0 failures.

File: atlas_description/robots/atlas_v5_sandia_hands.urdf.xacro (robot description, xacro)
@@ -12,9 +12,9 @@
   <gazebo>
     <!-- include plugin for the left sandia hand -->
-    <plugin name="leftsandia_hand_plugin" filename="libSandiaHandPlugin.so">
+    <plugin filename="SandiaHandPlugin" name="drcsim_gazebo_ros_plugins::SandiaHandPlugin">
       <side>left</side>
     </plugin>
     <!-- include plugin for the right sandia hand -->
-    <plugin name="right_sandia_hand_plugin" filename="libSandiaHandPlugin.so">
+    <plugin filename="SandiaHandPlugin" name="drcsim_gazebo_ros_plugins::SandiaHandPlugin">
       <side>right</side>
     </plugin>

File: sandia_hand_description/urdf/sandia_hand.gazebo.xacro (robot description, xacro)
@@ -158,18 +158,7 @@
           </noise>
         </camera>
-        <plugin filename="libgazebo_ros_multicamera.so" name="stereo_camera_controller">
-          <alwaysOn>true</alwaysOn>
-          <updateRate>0.0</updateRate>
-          <cameraName>sandia_hands/${parent}</cameraName>
-          <imageTopicName>image_raw</imageTopicName>
-          <cameraInfoTopicName>camera_info</cameraInfoTopicName>
-          <frameName>${side}_palm_left_camera_optical_frame</frameName>
-          <hackBaseline>${stereo_offset}</hackBaseline>
-          <distortionK1>0.0</distortionK1>
-          <distortionK2>0.0</distortionK2>
-          <distortionK3>0.0</distortionK3>
-          <distortionT1>0.0</distortionT1>
-          <distortionT2>0.0</distortionT2>
-        </plugin>
+        <!-- The Classic libgazebo_ros_multicamera.so ROS publisher has no
+             gz-sim equivalent here and was dropped (as for the MultiSense
+             head's cameras); the sensor itself still renders in gz. -->
       </sensor>
     </gazebo>
@@ -201,15 +190,7 @@
   </xacro:macro>
   <!-- end cameras -->
-  <xacro:macro name="sandia_hand_gazebo_controller" params="side">
-    <gazebo>
-      <plugin filename="libgazebo_ros_controller_manager.so" name="gazebo_ros_controller_manager">
-        <alwaysOn>true</alwaysOn>
-        <updateRate>1000.0</updateRate>
-      </plugin>
-    </gazebo>
-  </xacro:macro>
   <xacro:macro name="sandia_hand_tactile_sensors_gazebo" params="side parent" >
     <gazebo>
-      <plugin filename="libContactModelPlugin.so" name="sandia_contact_plugin">
+      <plugin filename="ContactModelPlugin" name="drcsim_gazebo_ros_plugins::ContactModelPlugin">
          <contact>
           <collision>${parent}::${parent}_collision_${side}_palm</collision>

File: sandia_hand_description/urdf/sandia_hand.urdf.xacro (robot description, xacro)
@@ -116,5 +116,5 @@
       </inertial>
     </link>
-    <joint name="${side}_f${idx}_base" type="fixed">
+    <joint name="${side}_f${idx}_base_joint" type="fixed">
       <parent link="${side}_palm"/>
       <child link="${side}_f${idx}_base"/>
@@ -148,15 +148,15 @@
       <limit lower="-${M_pi/2}" upper="${M_pi/2}" effort="28" velocity="${velocity_limit}"/>
     </joint>
-    <joint name="${side}_f${idx}_fixed_accel" type="fixed">
+    <joint name="${side}_f${idx}_fixed_accel_joint" type="fixed">
       <parent link="${side}_f${idx}_base"/>
       <child link="${side}_f${idx}_fixed_accel"/>
       <origin xyz="-0.05 0 0" rpy="0 0 0"/>
     </joint>
-    <joint name="${side}_f${idx}_1_accel" type="fixed">
+    <joint name="${side}_f${idx}_1_accel_joint" type="fixed">
       <parent link="${side}_f${idx}_1"/>
       <child link="${side}_f${idx}_1_accel"/>
       <origin xyz="0.03 0 0" rpy="-${M_pi/2} 0 0"/>
     </joint>
-    <joint name="${side}_f${idx}_2_accel" type="fixed">
+    <joint name="${side}_f${idx}_2_accel_joint" type="fixed">
       <parent link="${side}_f${idx}_2"/>
       <child link="${side}_f${idx}_2_accel"/>
@@ -201,5 +201,4 @@
     <xacro:finger side="${side}" idx="3" x="0.03995" y="${-0.04383*reflect}" z="0.014" r="0" p="-${M_pi/2 + thumb_angle}" yaw="${-(2.3562+thumb_angle)*reflect}" reflect="${reflect}" joint_type="${joint_type}"/>
     <!-- not needed unless simulating the hand by itself
-    <xacro:sandia_hand_gazebo_controller side="${side}" />
     -->
     <xacro:sandia_hand_gazebo side="${side}" />

File: sandia_hand_description/urdf/sandia_hand_simple_shapes.urdf.xacro (robot description, xacro)
@@ -214,5 +214,5 @@
       </inertial>
     </link>
-    <joint name="${side}_f${idx}_base" type="fixed">
+    <joint name="${side}_f${idx}_base_joint" type="fixed">
       <parent link="${side}_palm"/>
       <child link="${side}_f${idx}_base"/>
@@ -246,15 +246,15 @@
       <limit lower="-${M_pi/2}" upper="${M_pi/2}" effort="28" velocity="${velocity_limit}"/>
     </joint>
-    <joint name="${side}_f${idx}_fixed_accel" type="fixed">
+    <joint name="${side}_f${idx}_fixed_accel_joint" type="fixed">
       <parent link="${side}_f${idx}_base"/>
       <child link="${side}_f${idx}_fixed_accel"/>
       <origin xyz="-0.05 0 0" rpy="0 0 0"/>
     </joint>
-    <joint name="${side}_f${idx}_1_accel" type="fixed">
+    <joint name="${side}_f${idx}_1_accel_joint" type="fixed">
       <parent link="${side}_f${idx}_1"/>
       <child link="${side}_f${idx}_1_accel"/>
       <origin xyz="0.03 0 0" rpy="-${M_pi/2} 0 0"/>
     </joint>
-    <joint name="${side}_f${idx}_2_accel" type="fixed">
+    <joint name="${side}_f${idx}_2_accel_joint" type="fixed">
       <parent link="${side}_f${idx}_2"/>
       <child link="${side}_f${idx}_2_accel"/>
@@ -412,5 +412,4 @@
     <xacro:finger side="${side}" idx="3" x="0.03995" y="${-0.04383*reflect}" z="0.014" r="0" p="-${M_pi/2 + thumb_angle}" yaw="${-(2.3562+thumb_angle)*reflect}" reflect="${reflect}" joint_type="${joint_type}"/>
     <!-- not needed unless simulating the hand by itself
-    <xacro:sandia_hand_gazebo_controller side="${side}" />
     -->
     <xacro:sandia_hand_gazebo side="${side}" />
