Commit message: Fix every hand mount; Docker image (NVIDIA + CycloneDDS); modern skin; Robotiq option
Hands: the hand xacros used bare <insert_block> (ROS 1 xacro only), so
ROS 2 dropped every hand-mount transform and both palms sat on the wrist.
With that fixed, v4/v5 left mounts put the left hand inside the forearm
(v5's left-arm frames are rotated pi about z). Every left mount is now
derived as the mirror of the right one; test_hand_mounts.py checks all 17
*_hands variants by zero-pose FK. Screenshots confirm Sandia and Robotiq.

hands:=sandia|robotiq|none. Robotiq's closed finger loops can't be
simulated by DART; the state publishers get a URDF with those passive
joints fixed so RViz has full TF. iRobot's invalid inertia is fixed but it
still diverges in simulation, so it isn't offered.

skin:=modern (default): the spawned model gets PBR car-paint materials
(pearl panels, piano-black trim, graphite hands, red head).

docker/: Dockerfile (osrf/ros:jazzy-desktop-full + CycloneDDS, rosdep,
prebuilt workspace, NVIDIA all capabilities, PRIME offload switch), host
scripts build/run/sim/gui/teleop/shell/stop, in-container drcsim_sim/gui/
teleop/snapshot (Xvfb screenshots). With CycloneDDS the gz server renders
on the GPU without the FastDDS-era segfault.

File: atlas_description/robots/atlas_v3_irobot_hands.urdf.xacro (robot description, xacro)
@@ -6,5 +6,5 @@
   </xacro:irobot_hand>
   <xacro:irobot_hand side="left" parent="l_hand" reflect="-1">
-    <origin xyz="0.00179  0.09516 0.01176" rpy="-1.57079 0 0"/>
+    <origin xyz="-0.00179 0.09516 0.01176" rpy="1.57079 -0.00000 3.14159"/>
   </xacro:irobot_hand>
   <gazebo>

File: atlas_description/robots/atlas_v4_irobot_hands.urdf.xacro (robot description, xacro)
@@ -6,5 +6,5 @@
   </xacro:irobot_hand>
   <xacro:irobot_hand side="left" parent="l_hand" reflect="-1">
-    <origin xyz="0.00179  0.09516 0.01176" rpy="-1.57079 0 0"/>
+    <origin xyz="0.00179 -0.09516 0.03016" rpy="1.57079 -0.00000 -0.00000"/>
   </xacro:irobot_hand>
   <gazebo>

File: atlas_description/robots/atlas_v4_robotiq_hands.urdf.xacro (robot description, xacro)
@@ -5,5 +5,5 @@
   to mach the values in your actual robot. -->
   <xacro:robotiq_hand prefix="l_" parent="l_hand" reflect="-1">
-    <origin rpy="3.14159 3.14159 3.14159" xyz="-0.00125 0.17 0.01"/>
+    <origin xyz="0.00125 -0.17000 0.02840" rpy="0.00000 0.00000 3.14159"/>
   </xacro:robotiq_hand>
   <xacro:robotiq_hand prefix="r_" parent="r_hand" reflect="1">

File: atlas_description/robots/atlas_v4_sandia_hands.urdf.xacro (robot description, xacro)
@@ -6,5 +6,5 @@
   </xacro:sandia_hand>
   <xacro:sandia_hand side="left" parent="l_hand" reflect="-1" joint_type="revolute" thumb_angle="0">
-    <origin xyz="0.00179  0.13516 0.01176" rpy="0 0  1.57079"/>
+    <origin xyz="0.00179 -0.13516 0.03016" rpy="0.00000 0.00000 -1.57080"/>
   </xacro:sandia_hand>
   <xacro:include filename="$(find atlas_description)/urdf/atlas_v4.gazebo" />

File: atlas_description/robots/atlas_v5_irobot_hands.urdf.xacro (robot description, xacro)
@@ -5,14 +5,18 @@
     <origin xyz="-0.00179 -0.09516 0.01176" rpy="1.57079 0 0"/>
   </xacro:irobot_hand>
+  <!-- Left mount derived as the mirror image of the right one (v5's left-arm
+       frames are the right arm's rotated pi about z), using the hand's own
+       symmetry plane; checked by test/test_hand_mounts.py. The old values
+       put the left hand inside the forearm (see CLAUDE.md). -->
   <xacro:irobot_hand side="left" parent="l_hand" reflect="-1">
-    <origin xyz="0.00179  0.09516 0.01176" rpy="-1.57079 0 0"/>
+    <origin xyz="0.00179 -0.09516 0.01176" rpy="1.57079 -0.00000 -0.00000"/>
   </xacro:irobot_hand>
   <gazebo>
     <!-- plugin for right irobot hand -->
-    <plugin name="right_irobot_hand_plugin" filename="libIRobotHandPlugin.so">
+    <plugin filename="IRobotHandPlugin" name="drcsim_gazebo_ros_plugins::IRobotHandPlugin">
       <side>right</side>
     </plugin>
     <!-- plugin for left irobot hand -->
-    <plugin name="left_irobot_hand_plugin" filename="libIRobotHandPlugin.so">
+    <plugin filename="IRobotHandPlugin" name="drcsim_gazebo_ros_plugins::IRobotHandPlugin">
       <side>left</side>
     </plugin>

File: atlas_description/robots/atlas_v5_robotiq_hands.urdf.xacro (robot description, xacro)
@@ -4,6 +4,10 @@
   <!-- Set the initial hand position and orientation by changing 'rpy' and 'xyz'
   to mach the values in your actual robot. -->
+  <!-- Left mount derived as the mirror image of the right one (v5's left-arm
+       frames are the right arm's rotated pi about z), using the gripper's
+       own symmetry plane; checked by test/test_hand_mounts.py. The old
+       values put the left gripper inside the forearm (see CLAUDE.md). -->
   <xacro:robotiq_hand prefix="l_" parent="l_hand" reflect="-1">
-    <origin rpy="3.14159 3.14159 3.14159" xyz="-0.00125 0.17 0.01"/>
+    <origin xyz="0.00125 -0.17000 0.01000" rpy="0.00000 0.00000 3.14159"/>
   </xacro:robotiq_hand>
   <xacro:robotiq_hand prefix="r_" parent="r_hand" reflect="1">
@@ -12,5 +16,5 @@
   <gazebo>
     <!-- plugin for left RobotiQ hand -->
-    <plugin name="left_robotiq_hand_plugin" filename="libRobotiqHandPlugin.so">
+    <plugin filename="RobotiqHandPlugin" name="drcsim_gazebo_ros_plugins::RobotiqHandPlugin">
       <side>left</side>
       <kp_position>5.0</kp_position>
@@ -18,5 +22,5 @@
     </plugin>
     <!-- plugin for right RobotiQ hand -->
-    <plugin name="right_robotiq_hand_plugin" filename="libRobotiqHandPlugin.so">
+    <plugin filename="RobotiqHandPlugin" name="drcsim_gazebo_ros_plugins::RobotiqHandPlugin">
       <side>right</side>
       <kp_position>5.0</kp_position>

File: atlas_description/robots/atlas_v5_sandia_hands.urdf.xacro (robot description, xacro)
@@ -6,5 +6,9 @@
   </xacro:sandia_hand>
   <xacro:sandia_hand side="left" parent="l_hand" reflect="-1" joint_type="revolute" thumb_angle="0">
-    <origin xyz="0.00179  0.13516 0.01176" rpy="0 0  1.57079"/>
+    <!-- v5's left-arm frames are the right arm's rotated pi about z (l_arm_shz
+         rpy), so the mirror image of the right mount is x negated, y and
+         the rotation unchanged. Verified: fingers now point out past the
+         wrist, mirroring the right hand (see CLAUDE.md). -->
+    <origin xyz="0.00179 -0.13516 0.01176" rpy="0 0 -1.57079"/>
   </xacro:sandia_hand>
   <xacro:include filename="$(find atlas_description)/urdf/atlas_v5.gazebo" />

File: irobot_hand_description/urdf/irobot_hand.urdf.xacro (robot description, xacro)
@@ -324,5 +324,5 @@
   <!-- joint attaching parent link to irobot hand -->
   <joint name="${side}_irobot_hand_joint" type="fixed">
-    <insert_block name="origin"/>
+    <xacro:insert_block name="origin"/>
     <parent link="${parent}"/>
     <child link="${side}_base_link"/>
@@ -384,5 +384,8 @@
         -->
         <origin xyz="-0.002630 0.002396 0.021770" rpy="${pi/2} -${pi/2} 0"/>
-        <inertia ixx="2.420689e-6" ixy="-1.449042e-6" ixz="-7.74579e-7" iyy="1.196202e-6" iyz="1.90704e-7" izz="1.2736461e-6"/>
+        <!-- The CAD products of inertia gave principal moments (0.16, 1.11, 3.62)e-6
+             that violate the triangle inequality, which SDFormat rejects (the
+             whole robot then failed to spawn); the diagonal alone is valid. -->
+        <inertia ixx="2.420689e-6" ixy="0" ixz="0" iyy="1.196202e-6" iyz="0" izz="1.2736461e-6"/>
       </inertial>
     <xacro:proximal_link_collisions/>
@@ -457,5 +460,8 @@
         -->
         <origin xyz="-0.002630 0.002396 0.021770" rpy="${pi/2} -${pi/2} 0"/>
-        <inertia ixx="2.420689e-6" ixy="-1.449042e-6" ixz="-7.74579e-7" iyy="1.196202e-6" iyz="1.90704e-7" izz="1.2736461e-6"/>
+        <!-- The CAD products of inertia gave principal moments (0.16, 1.11, 3.62)e-6
+             that violate the triangle inequality, which SDFormat rejects (the
+             whole robot then failed to spawn); the diagonal alone is valid. -->
+        <inertia ixx="2.420689e-6" ixy="0" ixz="0" iyy="1.196202e-6" iyz="0" izz="1.2736461e-6"/>
       </inertial>
     <xacro:proximal_link_collisions/>
@@ -513,5 +519,8 @@
         -->
         <origin xyz="-0.002630 0.002396 0.021770" rpy="${pi/2} -${pi/2} 0"/>
-        <inertia ixx="2.420689e-6" ixy="-1.449042e-6" ixz="-7.74579e-7" iyy="1.196202e-6" iyz="1.90704e-7" izz="1.2736461e-6"/>
+        <!-- The CAD products of inertia gave principal moments (0.16, 1.11, 3.62)e-6
+             that violate the triangle inequality, which SDFormat rejects (the
+             whole robot then failed to spawn); the diagonal alone is valid. -->
+        <inertia ixx="2.420689e-6" ixy="0" ixz="0" iyy="1.196202e-6" iyz="0" izz="1.2736461e-6"/>
       </inertial>
     <xacro:proximal_link_collisions/>

File: robotiq_hand_description/urdf/robotiq_hand.urdf.xacro (robot description, xacro)
@@ -636,5 +636,5 @@
     <!-- joint attaching parent link to robotiq hand -->
     <joint name="${prefix}robotiq_hand_joint" type="fixed">
-      <insert_block name="origin"/>
+      <xacro:insert_block name="origin"/>
       <parent link="${parent}"/>
       <child link="${prefix}palm"/>

File: sandia_hand_description/urdf/sandia_hand.urdf.xacro (robot description, xacro)
@@ -194,5 +194,5 @@
       <parent link="${parent}"/>
       <child link="${side}_palm"/>
-      <insert_block name="origin" />
+      <xacro:insert_block name="origin"/>
     </joint>
     <xacro:finger side="${side}" idx="0" x="0.140" y="0.00000" z="0" r="0" p="0" yaw="${0.3*reflect}" reflect="${reflect}" joint_type="${joint_type}"/>

File: sandia_hand_description/urdf/sandia_hand_simple_shapes.urdf.xacro (robot description, xacro)
@@ -405,5 +405,5 @@
       <parent link="${parent}"/>
       <child link="${side}_palm"/>
-      <insert_block name="origin" />
+      <xacro:insert_block name="origin"/>
     </joint>
     <xacro:finger side="${side}" idx="0" x="0.140" y="0.00000" z="0" r="0" p="0" yaw="${0.3*reflect}" reflect="${reflect}" joint_type="${joint_type}"/>
